File: kiCad/Connectors.kicad_sch (KiCad schematic)
At the start: 3 parts, among them J1 Conn_01x02

Commit message: upd
Other:
- note added: "['at', '120', '100', '0']"
- note added: "['at', '90', '160', '0']"
Changed lines of the file:
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@@
     (date "2025-12-31")
   )
-  ;; === J1 Terminal Block ===
+  # === J1 Terminal Block ===
   (symbol (lib_id "Connector:Conn_01x02")
     (at 40 100 0)
@@
       (effects (font (size 1.27 1.27))))
   )
-  ;; === D1 SS34 Schottky ===
+  # === D1 SS34 Schottky ===
   (symbol (lib_id "Device:D_Schottky")
     (at 90 100 0)
@@
       (effects (font (size 1.27 1.27))))
   )
-  ;; === D2 SMAJ24CA TVS ===
+  # === D2 SMAJ24CA TVS ===
   (symbol (lib_id "Device:D_TVS")
     (at 90 140 0)
@@
       (effects (font (size 1.27 1.27))))
   )
-  ;; === Wires ===
-  (wire (pts (40 100) (70 100)))
-  (wire (pts (70 100) (90 100)))
-  (wire (pts (90 100) (120 100)))
-  ;; TVS to line
-  (wire (pts (90 140) (90 120)))
-  ;; === Net Labels ===
-  (net_label (at 120 100 0)
+  # === Wires ===
+  (wire (pts (xy 40 100) (xy 70 100)))
+  (wire (pts (xy 70 100) (xy 90 100)))
+  (wire (pts (xy 90 100) (xy 120 100)))
+  # TVS to line
+  (wire (pts (xy 90 140) (xy 90 120)))
+  # === Net Labels (as plain text) ===
+  (text (at 120 100 0)
     (text "VIN_RAW")
     (effects (font (size 1.27 1.27)))
   )
-  (net_label (at 90 160 0)
+  (text (at 90 160 0)
     (text "GND")
     (effects (font (size 1.27 1.27)))
   )
-  ;; === Junctions ===
+  # === Junctions ===
   (junction (at 90 100))
 )
