File: kiCad/buck.kicad_sch (KiCad schematic)
At the start: 7 parts

Commit message: upd
Parts:
- removed C1: 100nf, symbol Device:C
- removed C2: 470uf, symbol Device:C_Polarized
- removed D1: SS34, Diode_SMD:D_SMA, symbol Diode:SS34
- removed D2: D3V6, symbol Device:D_Zener
- removed D4: SS14, Diode_SMD:D_SMA, symbol Diode:SS14
- removed R2: R47K, symbol Device:R
- removed R3: R100K, symbol Device:R
- added C3: 100nf, symbol Device:C
- added C4: 33pf, symbol Device:C
- added C5: 10uF, symbol Device:C
- added C6: 100nF, symbol Device:C
- added D3: SS34, Diode_SMD:D_SMA, symbol Diode:SS34
- added L1: 2.2uH, symbol Device:L
- added R4: 124K, symbol Device:R
- added R5: 40.2K, symbol Device:R
- added U3: MP2451, Package_TO_SOT_SMD:SOT-23-6, symbol Regulator_Switching:LMR16006YQ
Connections:
- net GND_BUS: now also C5.2, C6.2, D3.2 (A), R5.2, U3.2 (GND)
- net V_BUCK_IN: now also C6.1, U3.4 (~{SHDN}), U3.5 (VIN)
- new net: C3.1, U3.1 (CB)
- new net: C3.2, D3.1 (K), L1.2, U3.6 (SW)
- new net: C4.2, R4.2, R5.1, U3.3 (FB)
- new net 3V3: C4.1, C5.1, L1.1, R4.1
Other:
- title: Power - Hold-up from RS485 -> (none)
