File: kiCad/Power.kicad_sch (KiCad schematic)
At the start: 7 parts

Commit message: Add Pcb
Parts:
- C1: footprint (none) -> Capacitor_SMD:C_0603_1608Metric; LCSC (none) -> C52711259
- C2: footprint (none) -> 123:CP_Elec_10x10; LCSC (none) -> C106703
- D1: footprint Diode_SMD:D_SMA -> 123:D_SOD-123; LCSC (none) -> C908669
- D2: footprint (none) -> Diode_SMD:D_SOD-123; LCSC (none) -> C173412
- D4: footprint Diode_SMD:D_SMA -> 123:D_SOD-123; LCSC (none) -> C2837270
- R2: footprint (none) -> Resistor_SMD:R_0603_1608Metric; LCSC (none) -> C17713
- R3: footprint (none) -> Resistor_SMD:R_0603_1608Metric; LCSC (none) -> C25741
Changed lines of the file:
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@@
 			)
 		)
-		(property "Footprint" ""
+		(property "Footprint" "Resistor_SMD:R_0603_1608Metric"
 			(at 69.342 54.61 90)
 			(effects
@@
 		)
 		(property "Description" "Resistor"
+			(at 71.12 54.61 0)
+			(effects
+				(font
+					(size 1.27 1.27)
+				)
+				(hide yes)
+			)
+		)
+		(property "LCSC" "C25741"
 			(at 71.12 54.61 0)
 			(effects
@@
 			)
 		)
-		(property "Footprint" "Diode_SMD:D_SMA"
+		(property "Footprint" "123:D_SOD-123"
 			(at 73.66 100.965 0)
 			(effects
@@
 		)
 		(property "Description" "40V 3A Schottky Diode, SMA"
+			(at 73.66 96.52 0)
+			(effects
+				(font
+					(size 1.27 1.27)
+				)
+				(hide yes)
+			)
+		)
+		(property "LCSC" "C908669"
 			(at 73.66 96.52 0)
 			(effects
@@
 			)
 		)
-		(property "Footprint" ""
+		(property "Footprint" "123:CP_Elec_10x10"
 			(at 78.4352 114.3 0)
 			(effects
@@
 		)
 		(property "Description" "Polarized capacitor"
+			(at 77.47 110.49 0)
+			(effects
+				(font
+					(size 1.27 1.27)
+				)
+				(hide yes)
+			)
+		)
+		(property "LCSC" "C106703"
 			(at 77.47 110.49 0)
 			(effects
@@
 			)
 		)
-		(property "Footprint" ""
+		(property "Footprint" "Resistor_SMD:R_0603_1608Metric"
 			(at 66.04 48.768 90)
 			(effects
@@
 		(property "Description" "Resistor"
 			(at 66.04 46.99 0)
+			(effects
+				(font
+					(size 1.27 1.27)
+				)
+				(hide yes)
+			)
+		)
+		(property "LCSC" "C17713"
+			(at 66.04 46.99 90)
 			(effects
 				(font
@@
 			)
 		)
-		(property "Footprint" "Diode_SMD:D_SMA"
+		(property "Footprint" "123:D_SOD-123"
 			(at 73.66 88.265 0)
 			(effects
@@
 		)
 		(property "Description" "40V 1A Schottky Diode, SMA"
+			(at 73.66 83.82 0)
+			(effects
+				(font
+					(size 1.27 1.27)
+				)
+				(hide yes)
+			)
+		)
+		(property "LCSC" "C2837270"
 			(at 73.66 83.82 0)
 			(effects
@@
 			)
 		)
-		(property "Footprint" ""
+		(property "Footprint" "Diode_SMD:D_SOD-123"
 			(at 83.82 54.61 0)
 			(effects
@@
 		(property "Description" "Zener diode"
 			(at 83.82 54.61 0)
+			(effects
+				(font
+					(size 1.27 1.27)
+				)
+				(hide yes)
+			)
+		)
+		(property "LCSC" "C173412"
+			(at 83.82 54.61 90)
 			(effects
 				(font
@@
 			)
 		)
-		(property "Footprint" ""
+		(property "Footprint" "Capacitor_SMD:C_0603_1608Metric"
 			(at 96.2152 114.3 0)
 			(effects
@@
 			(at 95.25 110.49 0)
 			(effects
+				(font
+					(size 1.27 1.27)
+				)
+				(hide yes)
+			)
+		)
+		(property "LCSC" "C52711259"
+			(at 95.25 110.49 0)
+			(effects
