File: kiCad/RS485.kicad_sch (KiCad schematic)
At the start: 1 part, among them U3 ADM2587E

Commit message: upd
Parts:
- removed U3: ADM2587E, symbol DriverRS485:ADM2587E
- added J1: Terminal_block_2p, symbol Connector_Generic:Conn_01x02
- added R1: 10R, symbol Device:R
- added U1: TVS2700DRV, Package_SON:WSON-6-1EP_2x2mm_P0.65mm_EP1x1.6mm, symbol Power_Protection:TVS2700DRV
Connections:
- new net GND_BUS: J1.2 (Pin_2), U1.1 (GND), U1.2 (GND), U1.3 (GND), U1.7 (GND)
- new net V_BUS: J1.1 (Pin_1), R1.2, U1.4 (IN), U1.5 (IN), U1.6 (IN)
- new net V_BUS_IN: R1.1
Other:
- company: Custom Electronics -> (none)
- title: RS485 Transceiver Stage -> Isolated RS485

Commit message: Add Pcb
Parts:
- removed U1: TVS2700DRV, Package_SON:WSON-6-1EP_2x2mm_P0.65mm_EP1x1.6mm, symbol Power_Protection:TVS2700DRV
- added D5: SMF24A, 123:D_SOD-123FL, symbol Diode:SMF24A
- J1: footprint (none) -> TerminalBlock_Phoenix:TerminalBlock_Phoenix_MKDS-1-2-3.81_1x02_P3.81mm_Horizontal; LCSC (none) -> C5188452
- R1: footprint (none) -> Resistor_SMD:R_1206_3216Metric; LCSC (none) -> C17901
Connections:
- net GND_BUS: now also D5.2 (A2)
- net V_BUS: now also D5.1 (A1)
Changed lines of the file:
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@@
 	(wire
 		(pts
-			(xy 64.77 71.12) (xy 46.99 71.12)
-		)
-		(stroke
-			(width 0)
-			(type default)
-		)
-	)
-	(wire
-		(pts
-			(xy 72.39 71.12) (xy 64.77 71.12)
-		)
-		(stroke
-			(width 0)
-			(type default)
-		)
-	)
-	(wire
-		(pts
-			(xy 64.77 86.36) (xy 64.77 87.63)
+			(xy 46.99 71.12) (xy 64.77 71.12)
+		)
+		(stroke
+			(width 0)
+			(type default)
+		)
+	)
+	(wire
+		(pts
+			(xy 64.77 82.55) (xy 64.77 87.63)
 		)
 		(stroke
@@
 	(wire
 		(pts
+			(xy 64.77 71.12) (xy 72.39 71.12)
+		)
+		(stroke
+			(width 0)
+			(type default)
+		)
+	)
+	(wire
+		(pts
 			(xy 81.28 71.12) (xy 80.01 71.12)
 		)
@@
 		(pts
 			(xy 46.99 71.12) (xy 46.99 80.01)
+		)
+		(stroke
+			(width 0)
+			(type default)
+		)
+	)
+	(wire
+		(pts
+			(xy 64.77 71.12) (xy 64.77 74.93)
 		)
 		(stroke
@@
 			)
 		)
-		(property "Footprint" ""
+		(property "Footprint" "TerminalBlock_Phoenix:TerminalBlock_Phoenix_MKDS-1-2-3.81_1x02_P3.81mm_Horizontal"
 			(at 41.91 80.01 0)
 			(effects
@@
 		)
 		(property "Description" "Generic connector, single row, 01x02, script generated (kicad-library-utils/schlib/autogen/connector/)"
+			(at 41.91 80.01 0)
+			(effects
+				(font
+					(size 1.27 1.27)
+				)
+				(hide yes)
+			)
+		)
+		(property "LCSC" "C5188452"
 			(at 41.91 80.01 0)
 			(effects
@@
 				(path "/11111111-aaaa-bbbb-cccc-000000000001/33333333-aaaa-bbbb-cccc-000000000003"
 					(reference "J1")
-					(unit 1)
-				)
-			)
-		)
-	)
-	(symbol
-		(lib_id "Power_Protection:TVS2700DRV")
-		(at 64.77 78.74 0)
-		(unit 1)
-		(exclude_from_sim no)
-		(in_bom yes)
-		(on_board yes)
-		(dnp no)
-		(fields_autoplaced yes)
-		(property "Reference" "U1"
-			(at 68.58 77.4699 0)
-			(effects
-				(font
-					(size 1.27 1.27)
-				)
-				(justify left)
-			)
-		)
-		(property "Value" "TVS2700DRV"
-			(at 68.58 80.0099 0)
-			(effects
-				(font
-					(size 1.27 1.27)
-				)
-				(justify left)
-			)
-		)
-		(property "Footprint" "Package_SON:WSON-6-1EP_2x2mm_P0.65mm_EP1x1.6mm"
-			(at 69.85 87.63 0)
-			(effects
-				(font
-					(size 1.27 1.27)
-				)
-				(hide yes)
-			)
-		)
-		(property "Datasheet" "http://www.ti.com/lit/ds/symlink/tvs2700.pdf"
-			(at 62.23 78.74 0)
-			(effects
-				(font
-					(size 1.27 1.27)
-				)
-				(hide yes)
-			)
-		)
-		(property "Description" "Flat-Clamp Surge Protection Device. 27Vrwm, WSON-6"
-			(at 64.77 78.74 0)
-			(effects
-				(font
-					(size 1.27 1.27)
-				)
-				(hide yes)
-			)
-		)
-		(pin "1"
-		)
-		(pin "2"
-		)
-		(pin "7"
-		)
-		(pin "4"
-		)
-		(pin "3"
-		)
-		(pin "5"
-		)
-		(pin "6"
-		)
-		(instances
-			(project ""
-				(path "/11111111-aaaa-bbbb-cccc-000000000001/33333333-aaaa-bbbb-cccc-000000000003"
-					(reference "U1")
 					(unit 1)
 				)
@@
 			)
 		)
-		(property "Footprint" ""
+		(property "Footprint" "Resistor_SMD:R_1206_3216Metric"
 			(at 76.2 69.342 90)
 			(effects
@@
 		(property "Description" "Resistor"
 			(at 76.2 71.12 0)
+			(effects
+				(font
+					(size 1.27 1.27)
+				)
+				(hide yes)
+			)
+		)
+		(property "LCSC" "C17901"
+			(at 76.2 71.12 90)
 			(effects
 				(font
@@
 					(unit 1)
 				)
+			)
+		)
+	)
+	(symbol
+		(lib_id "Diode:SMF24A")
+		(at 64.77 78.74 270)
+		(unit 1)
+		(exclude_from_sim no)
+		(in_bom yes)
+		(on_board yes)
+		(dnp no)
+		(fields_autoplaced yes)
+		(property "Reference" "D5"
+			(at 67.31 77.4699 90)
+			(effects
+				(font
+					(size 1.27 1.27)
+				)
+				(justify left)
+			)
+		)
+		(property "Value" "SMF24A"
+			(at 67.31 80.0099 90)
+			(effects
+				(font
+					(size 1.27 1.27)
+				)
+				(justify left)
+			)
+		)
+		(property "Footprint" "123:D_SOD-123FL"
+			(at 59.69 78.74 0)
+			(effects
+				(font
+					(size 1.27 1.27)
+				)
+				(hide yes)
+			)
+		)
+		(property "Datasheet" "https://www.vishay.com/doc?85881"
+			(at 64.77 77.47 0)
+			(effects
+				(font
+					(size 1.27 1.27)
+				)
+				(hide yes)
+			)
+		)
+		(property "Description" "200W unidirectional Transil Transient Voltage Suppressor, 24Vrwm, SMF"
+			(at 64.77 78.74 0)
+			(effects
+				(font
+					(size 1.27 1.27)
+				)
+				(hide yes)
+			)
+		)
+		(property "LCSC" "C6937186"
+			(at 64.77 78.74 90)
+			(effects
+				(font
+					(size 1.27 1.27)
+				)
+				(hide yes)
+			)
+		)
+		(pin "2"
+		)
+		(pin "1"
+		)
+		(instances
+			(project ""
+				(path "/11111111-aaaa-bbbb-cccc-000000000001/33333333-aaaa-bbbb-cccc-000000000003"
+					(reference "D5")
+					(unit 1)
+				)
