File: kiCad/Isolated_RS485_Bridge.kicad_pcb (KiCad board)
At the start: 2 copper layers, 22 x 45.2 mm, 25 parts, among them J1 Terminal_block_2p, J2 TC2030, U1 AP63203WU, U3 ESP32-S3-MINI-1

Commit message: update
Parts:
- moved U3 150.8 mm to (22.7, 24.8), turned to 0 degrees

Commit message: update
Parts:
- removed the R3 at (158.3, 59.2)
- removed REF** (x3): Fiducial_1mm_Mask3mm, Fiducial:Fiducial_1mm_Mask3mm
- C1, C3, C6: value 100nf -> 100nF
- C2: value 470uf -> 470uF
- D4: footprint 123:D_SOD-123 -> 123:D_SOD-123FL
- D6: footprint 123:LED_SK6805D-OPSCO_2.1x2.1mm -> 123:LED_WS2812B-2020_2x2.2mm
- R2: value R47K -> 47K
- R4, R5: value 2K2 -> 470
- U3: footprint RF_Module:ESP32-S2-MINI-1 -> PCM_Espressif:ESP32-S3-MINI-1
- moved U3 150.0 mm to (166.2, 68.7), turned to 180 degrees
- moved R4 1.06 mm to (157.4, 60.1)
- moved R5 1.06 mm to (155.9, 60.1)
- moved R2 0.92 mm to (157.9, 57.1)
- moved D2 0.90 mm to (155.9, 56.2)
- moved R3 0.60 mm to (156.7, 75.3)
- moved D6 0.27 mm to (156.9, 72.8), turned to -90 degrees
- moved D1 0.14 mm to (167.9, 52.2)
- moved D5 0.12 mm to (171.8, 50.7)
- moved C2 0.07 mm to (160.1, 47.4)
- renumbered R9 to R3
Connections:
- U3 pad 23: unconnected-(U3-USB_D--Pad23) -> /ESP32/D-
- U3 pad 24: /ESP32/D- -> /ESP32/D+
- U3 pad 25: /ESP32/D+ -> unconnected-(U3-IO21-Pad25)
Routing:
- net /Buck/V_BUCK_IN: track 8.11 -> 10.0 mm
- net /Buck/3V3: track 45.1 -> 46.5 mm
- net /ESP32/BUS_TX: track 3.89 -> 2.68 mm
- net /ESP32/BUS_RX: track 5.34 -> 4.39 mm
- net /Buck/SW: track 5.42 -> 4.56 mm
- net /Power/V_BUS_IN: track 13.2 -> 13.9 mm
- net /ESP32/D-: track 16.7 -> 17.4 mm
- net /ESP32/D+: track 16.8 -> 17.4 mm
- net /Buck/GND: vias 2 -> 16

Commit message: first working version with last kicad design
Parts:
- removed D5: SMF24A, 123:D_SOD-123FL
- removed D6: WS2812B-2020, 123:LED_WS2812B-2020_2x2.2mm
- removed J2: TC2030, Connector:Tag-Connect_TC2030-IDC-NL_2x03_P1.27mm_Vertical
- removed R3: 10K, Resistor_SMD:R_0603_1608Metric
- removed R4, R5: 470, Resistor_SMD:R_0603_1608Metric
- added A1: B, TerminalBlock_Phoenix:TerminalBlock_Phoenix_MKDS-1-2-3.81_1x02_P3.81mm_Horizontal, F.Cu at (171.8, 45.3)
- added C8: 22uF, Capacitor_SMD:C_0805_2012Metric, F.Cu at (167.9, 58.6)
- added D3: SS14, 123:D_SOD-323HE, F.Cu at (154.9, 81.8)
- added PS1: MEE1S0303SC, Converter_DCDC:Converter_DCDC_Murata_MEE1SxxxxSC_THT, F.Cu at (157.2, 59.0)
- added U2: AP63203WU, Package_TO_SOT_SMD:TSOT-23-6, F.Cu at (157.2, 62.5)
- added U4: π122U31, Package_SO:SOIC-8_3.9x4.9mm_P1.27mm, F.Cu at (171.7, 65.7)
- added U5: THVD2450DR, Package_SO:SOIC-8_3.9x4.9mm_P1.27mm, F.Cu at (171.6, 58.0)
- C1: value 100nF -> 470uF; footprint Capacitor_SMD:C_0603_1608Metric -> 123:CP_Elec_10x10
- C2: value 470uF -> 100nF; footprint 123:CP_Elec_10x10 -> Capacitor_SMD:C_0603_1608Metric
- D1: value SS34 -> SMF24A; footprint 123:D_SOD-123 -> 123:D_SOD-123FL
- D2: value D3V6 -> WS2812B-2020; footprint Diode_SMD:D_SOD-123 -> 123:LED_WS2812B-2020_2x2.2mm
- D4: footprint 123:D_SOD-123FL -> 123:D_SOD-323HE
- J1: value Terminal_block_2p -> TC2030; footprint TerminalBlock_Phoenix:TerminalBlock_Phoenix_MKDS-1-2-3.81_1x02_P3.81mm_Horizontal -> Connector:Tag-Connect_TC2030-IDC-NL_2x03_P1.27mm_Vertical
- R2: value 47K -> 10K
- U1: value AP63203WU -> ESP32-S3-MINI-1; footprint Package_TO_SOT_SMD:TSOT-23-6 -> PCM_Espressif:ESP32-S3-MINI-1
- U3: value ESP32-S3-MINI-1 -> π122U31; footprint PCM_Espressif:ESP32-S3-MINI-1 -> Package_SO:SOIC-8_3.9x4.9mm_P1.27mm
- moved J1 34.9 mm to (156.5, 76.6), turned to 90 degrees
- moved R2 27.2 mm to (157.0, 84.3), turned to 0 degrees
- moved D2 25.6 mm to (157.2, 81.8), turned to -90 degrees
- moved C5 23.2 mm to (155.4, 71.3), turned to -90 degrees
- moved U1 20.6 mm to (166.5, 77.7), turned to 180 degrees
- moved C6 19.1 mm to (157.1, 71.1), turned to 90 degrees
- moved C4 16.1 mm to (159.8, 67.7), turned to 90 degrees
- moved C2 15.6 mm to (154.7, 62.0), turned to -90 degrees
- moved L1 14.7 mm to (156.6, 67.0), turned to 90 degrees
- moved C1 12.9 mm to (160.1, 47.5), turned to 90 degrees
- moved C3 10.9 mm to (159.6, 64.2), turned to 90 degrees
- moved D4 10.5 mm to (167.9, 50.6), turned to 0 degrees
- moved U3 3.08 mm to (166.3, 65.6), turned to 90 degrees
- moved R1 2.36 mm to (171.9, 50.7)
- moved D1 1.61 mm to (169.3, 53.0), turned to 0 degrees
Connections:
- C1 pad 1: /Buck/V_BUCK_IN -> /V_BUCK_IN
- C1 pad 2: /Buck/GND -> /GND_BUS
- C2 pad 1: /Buck/V_BUCK_IN -> /V_BUCK_IN
- C2 pad 2: /Buck/GND -> /GND_BUS
- C3 pad 1: /Buck/SW -> /SW
- C3 pad 2: /Buck/BST -> /BST
- C4 pad 1: /Buck/3V3 -> /3V3
- C4 pad 2: /Buck/GND -> /GND_BUS
- C5 pad 1: /Buck/3V3 -> /3V3
- C5 pad 2: /Buck/GND -> /GND_BUS
- C6 pad 1: /Buck/3V3 -> /GND_BUS
- C6 pad 2: /Buck/GND -> /3V3
- D1 pad 1: /Buck/V_BUCK_IN -> /V_BUCK_IN
- D1 pad 2: /Power/V_BUS_IN -> /GND_BUS
- D2 pad 1: /ESP32/BUS_IO -> unconnected-(D2-DOUT-Pad1)
- D2 pad 2: /Buck/GND -> /GND_BUS
- D4 pad 1: /Buck/V_BUCK_IN -> /V_BUCK_IN
- D4 pad 2: /ESP32/USB_5V -> Net-(D4-A)
- J1 pad 1: /RS485/V_BUS -> /5V_USB
- J1 pad 2: /Buck/GND -> /5V_USB
- L1 pad 1: /Buck/3V3 -> /3V3
- L1 pad 2: /Buck/SW -> /SW
- R1 pad 1: /Power/V_BUS_IN -> Net-(D4-A)
- R1 pad 2: /RS485/V_BUS -> /V_BUS
- R2 pad 1: /Power/V_BUS_IN -> /3V3
- R2 pad 2: /ESP32/BUS_IO -> /Reset
- U1 pad 1: /Buck/3V3 -> /GND_BUS
- U1 pad 2: /Buck/V_BUCK_IN -> /GND_BUS
- U1 pad 3: /Buck/V_BUCK_IN -> /3V3
- U1 pad 4: /Buck/GND -> unconnected-(U1-IO0-Pad4)
- U1 pad 5: /Buck/SW -> unconnected-(U1-IO1-Pad5)
- U1 pad 6: /Buck/BST -> unconnected-(U1-IO2-Pad6)
- U3 pad 1: /Buck/GND -> /3V3
- U3 pad 2: /Buck/GND -> /ESP32_RX
- U3 pad 3: /Buck/3V3 -> /ESP32_DE_RE
- U3 pad 4: unconnected-(U3-IO0-Pad4) -> /GND_BUS
- U3 pad 5: unconnected-(U3-IO1-Pad5) -> /GND_ISO
- U3 pad 6: unconnected-(U3-IO2-Pad6) -> /DE_RE_ISO
- U3 pad 7: unconnected-(U3-IO3-Pad7) -> /RX_ISO
- U3 pad 8: unconnected-(U3-IO4-Pad8) -> /3V3_ISO
Routing:
- net /3V3: track 0.00 -> 72.7 mm, vias 0 -> 4
- net /V_BUCK_IN: track 0.00 -> 52.4 mm, vias 0 -> 2
- net /Buck/3V3: track 46.5 -> 0.00 mm, vias 5 -> 0
- net /3V3_ISO: track 0.00 -> 19.3 mm
- net /ESP32/D+: track 17.4 -> 0.00 mm, vias 2 -> 0
- net /ESP32/D-: track 17.4 -> 0.00 mm, vias 2 -> 0
- net /Power/V_BUS_IN: track 13.9 -> 0.00 mm, vias 2 -> 0
- net /ESP32/USB_5V: track 13.9 -> 0.00 mm, vias 2 -> 0
- net /D+: track 0.00 -> 13.8 mm, vias 0 -> 2
- net /D-: track 0.00 -> 13.8 mm, vias 0 -> 2
- net /V_BUS: track 0.00 -> 11.4 mm
- net /Buck/V_BUCK_IN: track 10.0 -> 0.00 mm
- net /DE_RE_ISO: track 0.00 -> 7.17 mm
- net /RX_ISO: track 0.00 -> 6.11 mm
- net /SW: track 0.00 -> 5.40 mm
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- added copper zone on B.Cu, net /GND_BUS
- added copper zone on F.Cu, net /GND_BUS
- added copper zone on B.Cu, net /GND_ISO
- added copper zone on F.Cu, net /GND_ISO
- removed copper zone on F.Cu, net /Buck/3V3
- removed copper zone on B.Cu, net /Buck/GND
- removed copper zone on F.Cu, net /Buck/GND
- removed copper zone on F.Cu, net /Buck/V_BUCK_IN
- removed copper zone on F.Cu, net /ESP32/BUS_IO
- removed copper zone on F.Cu, net /Power/V_BUS_IN
- removed copper zone on F.Cu, net /RS485/V_BUS
Other:
- board size 22 x 45.2 mm -> 22 x 53.5 mm
- board text added: "A⁺²⁴"
- board text added: "B⏚"
