File: kiCad/Isolated_RS485_Bridge.kicad_sch (KiCad schematic)
At the start: 0 parts

Commit message: upd
Other:
- removed sheet Connectors
- added sheet Buck (buck.kicad_sch)
- sheet ESP32 ports: added 3V3, BUS_IO, GND_BUS, USB_5V; removed none
- sheet Power ports: added BUS_IO, GND_BUS, USB_5V, V_BUCK_IN, V_BUS_IN; removed none
- sheet RS485 ports: added GND_BUS, V_BUS_IN; removed none
- company: Custom Electronics -> (none)
- title: Isolated RS485 WiFi Bridge -> Isolated RS485 Bridge

Commit message: first working version with last kicad design
Parts:
- added A1: B, TerminalBlock_Phoenix:TerminalBlock_Phoenix_MKDS-1-2-3.81_1x02_P3.81mm_Horizontal, symbol Connector_Generic:Conn_01x02
- added C1: 470uF, 123:CP_Elec_10x10, symbol Device:C_Polarized
- added C2, C3, C6: 100nF, Capacitor_SMD:C_0603_1608Metric, symbol Device:C
- added C4, C5, C8: 22uF, Capacitor_SMD:C_0805_2012Metric, symbol Device:C
- added D1: SMF24A, 123:D_SOD-123FL, symbol Diode:SMF24A
- added D2: WS2812B-2020, 123:LED_WS2812B-2020_2x2.2mm, symbol LED:WS2812B-2020
- added D3: SS14, 123:D_SOD-323HE, symbol Diode:SS14
- added D4: SS14, 123:D_SOD-323HE, symbol Diode:SS34
- added J1: TC2030, Connector:Tag-Connect_TC2030-IDC-NL_2x03_P1.27mm_Vertical, symbol Connector:TC2030
- added L1: 4.7uH, Inductor_SMD:L_Bourns-SRN4018, symbol Device:L
- added PS1: MEE1S0303SC, Converter_DCDC:Converter_DCDC_Murata_MEE1SxxxxSC_THT, symbol Converter_DCDC:MEE1S0303SC
- added R1: 10R, Resistor_SMD:R_1206_3216Metric, symbol Device:R
- added R2: 10K, Resistor_SMD:R_0603_1608Metric, symbol Device:R
- added U1: ESP32-S3-MINI-1, PCM_Espressif:ESP32-S3-MINI-1, symbol RF_Module:ESP32-S3-MINI-1
- added U2: AP63203WU, Package_TO_SOT_SMD:TSOT-23-6, symbol Regulator_Switching:AP63203WU
- added U3, U4: π122U31, Package_SO:SOIC-8_3.9x4.9mm_P1.27mm, symbol Isolator:ISO7321C
- added U5: THVD2450DR, Package_SO:SOIC-8_3.9x4.9mm_P1.27mm, symbol Interface_UART:MAX485E
Connections:
- new net: D4.2 (A), R1.1
- new net 3V3: C4.1, C5.1, C6.2, D2.4 (VDD), L1.1, PS1.2 (+Vin), R2.1, U1.3 (3V3), U2.1 (FB), U3.1 (VCC1), U4.1 (VCC1)
- new net 3V3_ISO: C8.1, PS1.4 (+Vout), U3.8 (VCC2), U4.8 (VCC2), U5.8 (VCC)
- new net 5V_USB: D3.2 (A), J1.1, J1.2
- new net BST: C3.2, U2.6 (BST)
- new net D+: J1.4, U1.24 (USB_D+)
- new net D-: J1.3, U1.23 (USB_D-)
- new net DE_RE_ISO: U3.6 (OUTB), U5.2 (~{RE}), U5.3 (DE)
- new net ESP32_DE_RE: U1.22 (IO18), U3.3 (INB)
- new net ESP32_RX: U1.25 (IO21), U3.2 (OUTA)
- new net ESP32_TX: U1.16 (IO12), U4.3 (INB)
- new net GND_BUS: A1.2 (Pin_2), C1.2, C2.2, C4.2, C5.2, C6.1, D1.2 (A2), D2.2 (VSS), J1.5, J1.6, PS1.1 (-Vin), U1.1 (GND), U1.2 (GND), U1.42 (GND), U1.43 (GND), U1.46 (GND), U1.47 (GND), U1.48 (GND), U1.49 (GND), U1.50 (GND), U1.51 (GND), U1.52 (GND), U1.53 (GND), U1.54 (GND), U1.55 (GND), U1.56 (GND), U1.57 (GND), U1.58 (GND), U1.59 (GND), U1.60 (GND), U1.61 (GND), U1.62 (GND), U1.63 (GND), U1.64 (GND), U1.65 (GND), U2.4 (GND), U3.4 (GND1), U4.4 (GND1), U5.7 (B)
- new net GND_ISO: C8.2, PS1.3 (-Vout), U3.5 (GND2), U4.5 (GND2), U5.5 (GND)
- new net LED: D2.3 (DIN), U1.41 (IO45)
- new net RX_ISO: U3.7 (INA), U5.1 (RO)
- new net Reset: R2.2, U1.45 (EN)
- new net SW: C3.1, L1.2, U2.5 (SW)
- new net TX_ISO: U4.6 (OUTB), U5.4 (DI)
- new net V_BUCK_IN: C1.1, C2.1, D1.1 (A1), D3.1 (K), D4.1 (K), U2.2 (EN), U2.3 (IN)
- new net V_BUS: A1.1 (Pin_1), R1.2, U5.6 (A)
- no-connect marks 0 -> 36
Other:
- removed sheet Buck
- removed sheet ESP32
- removed sheet Power
- removed sheet RS485
